File: RP2350.kicad_sch (KiCad schematic)
At the start: 42 parts, among them U1 RP2350B

Commit message: Adding PGA2350 and RM2 module KiCad footprints and symbols
Parts:
- removed C1, C10, C11, C12, C13, C14, C15, C16, C17, C18, C19, C2, C20, C3, C4, C5, C6, C7, C8, C9: C_Small, symbol Device:C_Small
- removed R10, R11, R12, R13, R14, R15, R16, R17, R18, R19, R20, R3, R4, R5, R6, R7, R8, R9: R_Small, symbol Device:R_Small
- removed U1: RP2350B, Package_DFN_QFN:QFN-80-1EP_10x10mm_P0.4mm_EP3.4x3.4mm, symbol MCU_RaspberryPi:RP2350B
- removed XTAL1: SIT1602AC-22-33E-12.000000E, SON4_SIT1602-2_SIT, symbol SIT1602AC_22_33E_12:SIT1602AC-22-33E-12.000000E
- added BT1: Battery, symbol Device:Battery
- added D1, D2: LED_Small, symbol Device:LED_Small
- added L1: L_Small, symbol Device:L_Small
- added SW1: SW_SPST, symbol Switch:SW_SPST
- added U1: (no value), GP2040-CE_Library:PGA2350, symbol GP2040-CE_Library:PGA2350
- added U2: (no value), GP2040-CE_Library:RM2, symbol GP2040-CE_Library:RM2
- added U3: LiPo Amigo Pro, symbol GP2040-CE_Library:LiPo_Amigo_Pro
- R1: value 1k -> 10k
- R2: value R_Small -> 470R
Connections:
- net GND: now also D2.1 (K), U1.0 (GND), U1.1 (GND), U1.48 (GND), U1.49 (GND), U1.50 (GND), U1.51 (GND), U2.1 (GND), U2.11 (GND), U2.15 (GND), U2.21 (GND), U2.4 (GND), U2.7 (GND), U3.1 (GND), U3.5 (GND), U3.8 (GND); no longer R1.2
- net at R2.1: now also U2.6 (gSPI_Data_Out)
- net gSPI_Data_In: now reaches R2.2
- net gSPI_Data_In: now also R1.2, U1.24 (GP24), U2.5 (gSPI_Data_In)
- net IOVDD: no longer names the net of R1.1
- net IOVDD: now also U2.10 (nIRQ)
- new net +3.3V: L1.1, U1.60 (3v3)
- new net +5V: U1.61 (VBUS), U3.6 (VSYS)
- new net BATN: BT1.2 (-), U3.14 (BATN)
- new net BATP: BT1.1 (+), U3.13 (BATP)
- new net CLED: D1.1 (K), U3.3 (ChargeLED)
- new net DM: U1.55 (USB_DM), U3.12 (DM)
- new net DP: U1.54 (USB_DP), U3.11 (DP)
- new net PLED: D2.2 (A), U3.4 (PowerLED)
- new net PSwitchA: SW1.1 (A), U3.9 (PSwitch_A)
- new net PSwitchB: SW1.2 (B), U3.10 (PSwitch_B)
- new net VBUS: D1.2 (A), U3.2 (USB_5V)
- new net VDDBAT: L1.2, U2.14 (VDDIO), U2.16 (VIN)
- new net WL_GPIO0: U2.8 (GPIO0)
- new net WL_GPIO1: U2.18 (GPIO1)
- new net WL_GPIO2: U2.17 (GPIO2)
- new net Wi-Fi_ON: U2.12 (Wi-Fi_ON), U2.13 (BT_ON)
- new net gSPI_CS: U1.25 (GP25), U2.9 (gSPI_CS)
- new net gSPI_SCLK: U1.29 (GP29), U2.3 (gSPI_SCLK)
- no-connect marks 0 -> 4
Other:
- removed sheet USB-C
